File: hardware/heating-controller/heating-controller.kicad_sch (KiCad schematic)
At the start: 38 parts, among them J1 Temperature_probes, J2 LilyGo T-Display S3, J3 Power connector, J4 USER_LED, J5 EXT_LED, K1 FINDER-32.21-x000, Q1 AO3400A, Q2 AO3400A, U1 MAX6682, U2 MAX6682, U3 H11AA1

Commit message: MAX682 hardware
Parts:
- added R14, R15: 10k, Resistor_SMD:R_0603_1608Metric, symbol Device:R
- R4, R5: value 15k -> 1.2k
Connections:
- net +3.3V: now also R14.2, R15.2
- net ~{EXT_CS}: now also R15.1
- net ~{LIM_CS}: now also R14.1
Changed lines of the file:
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@@
   (junction (at 227.965 159.385) (diameter 0) (color 0 0 0 0)
   )
+  (junction (at 122.555 104.14) (diameter 0) (color 0 0 0 0)
+  )
   (junction (at 27.94 92.075) (diameter 0) (color 0 0 0 0)
   )
@@
   (junction (at 230.505 145.415) (diameter 0) (color 0 0 0 0)
   )
+  (junction (at 125.095 111.76) (diameter 0) (color 0 0 0 0)
+  )
   (junction (at 88.265 140.97) (diameter 0) (color 0 0 0 0)
   )
   (junction (at 153.67 177.165) (diameter 0) (color 0 0 0 0)
   )
+  (junction (at 125.095 92.71) (diameter 0) (color 0 0 0 0)
+  )
   (junction (at 217.805 145.415) (diameter 0) (color 0 0 0 0)
   )
   (junction (at 230.505 130.175) (diameter 0) (color 0 0 0 0)
   )
+  (junction (at 122.555 85.09) (diameter 0) (color 0 0 0 0)
+  )
   (junction (at 27.94 99.695) (diameter 0) (color 0 0 0 0)
   )
@@
     (stroke (width 0) (type default))
   )
-  (wire (pts (xy 122.555 104.14) (xy 122.555 100.965))
+  (wire (pts (xy 122.555 100.965) (xy 122.555 104.14))
     (stroke (width 0) (type default))
   )
@@
     (stroke (width 0) (type default))
   )
+  (wire (pts (xy 125.095 92.71) (xy 128.905 92.71))
+    (stroke (width 0) (type default))
+  )
   (wire (pts (xy 124.46 145.415) (xy 129.54 145.415))
     (stroke (width 0) (type default))
@@
     (stroke (width 0) (type default))
   )
+  (wire (pts (xy 125.095 104.14) (xy 122.555 104.14))
+    (stroke (width 0) (type default))
+  )
   (wire (pts (xy 155.575 147.32) (xy 165.735 147.32))
     (stroke (width 0) (type default))
@@
     (stroke (width 0) (type default))
   )
+  (wire (pts (xy 128.905 111.76) (xy 125.095 111.76))
+    (stroke (width 0) (type default))
+  )
+  (wire (pts (xy 119.38 92.71) (xy 125.095 92.71))
+    (stroke (width 0) (type default))
+  )
   (wire (pts (xy 46.355 77.47) (xy 46.355 72.39))
     (stroke (width 0) (type default))
@@
     (stroke (width 0) (type default))
   )
+  (wire (pts (xy 125.095 111.76) (xy 119.38 111.76))
+    (stroke (width 0) (type default))
+  )
   (wire (pts (xy 27.94 90.17) (xy 27.94 92.075))
     (stroke (width 0) (type default))
@@
     (stroke (width 0) (type default))
   )
+  (wire (pts (xy 122.555 85.09) (xy 125.095 85.09))
+    (stroke (width 0) (type default))
+  )
   (wire (pts (xy 84.455 87.63) (xy 84.455 90.17))
     (stroke (width 0) (type default))
@@
     (effects (font (size 1.27 1.27)) (justify left bottom))
   )
-  (label "~{EXT_CS}" (at 119.38 111.76 0) (fields_autoplaced)
+  (label "~{EXT_CS}" (at 128.905 111.76 0) (fields_autoplaced)
     (effects (font (size 1.27 1.27)) (justify left bottom))
   )
@@
     (effects (font (size 1.27 1.27)) (justify left bottom))
   )
-  (label "~{LIM_CS}" (at 119.38 92.71 0) (fields_autoplaced)
+  (label "~{LIM_CS}" (at 128.905 92.71 0) (fields_autoplaced)
     (effects (font (size 1.27 1.27)) (justify left bottom))
   )
@@
   (symbol (lib_id "Device:R") (at 98.425 106.68 90) (unit 1)
     (in_bom yes) (on_board yes) (dnp no) (fields_autoplaced)
-    (property "Reference" "R5" (at 98.425 101.9642 90)
-      (effects (font (size 1.27 1.27)))
-    )
-    (property "Value" "15k" (at 98.425 104.5011 90)
+    (property "Reference" "R5" (at 98.425 101.5197 90)
+      (effects (font (size 1.27 1.27)))
+    )
+    (property "Value" "1.2k" (at 98.425 103.9439 90)
       (effects (font (size 1.27 1.27)))
     )
@@
   (symbol (lib_id "Device:R") (at 98.425 87.63 90) (unit 1)
     (in_bom yes) (on_board yes) (dnp no) (fields_autoplaced)
-    (property "Reference" "R4" (at 98.425 82.9142 90)
-      (effects (font (size 1.27 1.27)))
-    )
-    (property "Value" "15k" (at 98.425 85.4511 90)
+    (property "Reference" "R4" (at 98.425 82.4697 90)
+      (effects (font (size 1.27 1.27)))
+    )
+    (property "Value" "1.2k" (at 98.425 84.8939 90)
       (effects (font (size 1.27 1.27)))
     )
@@
         (path "/4350e48f-c301-4acf-ab4d-ada5edc4f2b0"
           (reference "R9") (unit 1)
+        )
+      )
+    )
+  )
+  (symbol (lib_id "Device:R") (at 125.095 107.95 180) (unit 1)
+    (in_bom yes) (on_board yes) (dnp no) (fields_autoplaced)
+    (property "Reference" "R15" (at 126.873 106.7379 0)
+      (effects (font (size 1.27 1.27)) (justify right))
+    )
+    (property "Value" "10k" (at 126.873 109.1621 0)
+      (effects (font (size 1.27 1.27)) (justify right))
+    )
+    (property "Footprint" "Resistor_SMD:R_0603_1608Metric" (at 126.873 107.95 90)
+      (effects (font (size 1.27 1.27)) hide)
+    )
+    (property "Datasheet" "~" (at 125.095 107.95 0)
+      (effects (font (size 1.27 1.27)) hide)
+    )
+    (pin "1")
+    (pin "2")
+    (instances
+      (project "heating-controller"
+        (path "/4350e48f-c301-4acf-ab4d-ada5edc4f2b0"
+          (reference "R15") (unit 1)
         )
       )
@@
         )
       )
+    )
+  )
+  (symbol (lib_id "Device:R") (at 125.095 88.9 180) (unit 1)
+    (in_bom yes) (on_board yes) (dnp no) (fields_autoplaced)
+    (property "Reference" "R14" (at 126.873 87.6879 0)
+      (effects (font (size 1.27 1.27)) (justify right))
+    )
+    (property "Value" "10k" (at 126.873 90.1121 0)
+      (effects (font (size 1.27 1.27)) (justify right))
+    )
+    (property "Footprint" "Resistor_SMD:R_0603_1608Metric" (at 126.873 88.9 90)
+      (effects (font (size 1.27 1.27)) hide)
+    )
+    (property "Datasheet" "~" (at 125.095 88.9 0)
+      (effects (font (size 1.27 1.27)) hide)
+    )
+    (pin "1")
+    (pin "2")
+    (instances
+      (project "heating-controller"
+        (path "/4350e48f-c301-4acf-ab4d-ada5edc4f2b0"
+          (reference "R14") (unit 1)
+        )
+      )
